Commit message: Changed some inertial settings

File: src/myrobot_gazebo/urdf/myrobot_wheel.urdf.xacro (robot description, xacro)
@@ -4,7 +4,8 @@
 		<link name="${wheel_prefix}_wheel">
 			<inertial>
-				<mass value="2" />
-				<origin xyz="0.0 0.0 0.0" rpy="0 ${M_PI/2} ${M_PI/2}"/>
-				<inertia ixx="0.1" ixy="0.0" ixz="0.0" iyy="0.1" iyz="0.0" izz="0.1"/>
+				<mass value="1.5" />
+				<!-- <origin xyz="0.0 0.0 0.0" rpy="0 ${M_PI/2} ${M_PI/2}"/> -->
+				<origin xyz="0.0 0.0 0.0" rpy="0 0 0"/>
+				<inertia ixx="0.15" ixy="0.0" ixz="0.0" iyy="0.15" iyz="0.0" izz="0.15"/>
 			</inertial>
 			<visual name="${wheel_prefix}_wheel_visual">
@@ -34,6 +35,6 @@
 		</link>
 		<gazebo reference="${wheel_prefix}_wheel">
-			<mu1 value="1.0"/>
-			<mu2 value="1.0"/>
+			<mu1 value="1"/>
+			<mu2 value="1"/>
 			<kp value="10000000.0" />
 			<kd value="1.0" />

Commit message: Reduced wheel inertia and sidewards friction to improve turning

File: src/myrobot_gazebo/urdf/myrobot_wheel.urdf.xacro (robot description, xacro)
@@ -7,5 +7,5 @@
 				<!-- <origin xyz="0.0 0.0 0.0" rpy="0 ${M_PI/2} ${M_PI/2}"/> -->
 				<origin xyz="0.0 0.0 0.0" rpy="0 0 0"/>
-				<inertia ixx="0.15" ixy="0.0" ixz="0.0" iyy="0.15" iyz="0.0" izz="0.15"/>
+				<inertia ixx="0.005" ixy="0.0" ixz="0.0" iyy="0.005" iyz="0.0" izz="0.005"/>
 			</inertial>
 			<visual name="${wheel_prefix}_wheel_visual">
