Commit message: Added parameter to specify use of drive controller or skid steer plugin

File: src/myrobot_gazebo/urdf/myrobot.urdf.xacro (robot description, xacro)
@@ -2,18 +2,20 @@
 <robot name="myrobot"
     xmlns:xacro="http://www.ros.org/wiki/xacro">
-    <!-- PLUGINS -->
-    <xacro:include filename="$(find myrobot_gazebo)/urdf/myrobot.gazebo" />
     <!-- SUB-COMPONENTS -->
     <xacro:include filename="$(find myrobot_gazebo)/urdf/myrobot_wheel.urdf.xacro" />
     <!-- PROPERTIES -->
     <xacro:property name="M_PI" value="3.14159"/>
+    <xacro:property name="chassis_height" value="0.12" />
+    <xacro:property name="chassis_length" value="0.4" />
+    <xacro:property name="chassis_width" value="0.25" />
     <xacro:property name="wheel_width" value="0.06" />
     <xacro:property name="wheel_rad" value="0.1" />
     <xacro:property name="wheel_forward_offset" value="0.13" />
-    <xacro:property name="wheel_left_offset" value="0.15" />
+    <xacro:property name="wheel_left_offset" value="${chassis_width/2 + 0.05}" />
     <xacro:property name="wheel_friction" value="0.3" />
-    <xacro:property name="chassis_height" value="0.12" />
-    <xacro:property name="chassis_length" value="0.4" />
-    <xacro:property name="chassis_width" value="0.22" />
+    <xacro:property name="use_drive_controller" value="true" />
+    <!-- PLUGINS -->
+    <xacro:include filename="$(find myrobot_gazebo)/urdf/myrobot.gazebo.xacro" />
+    <!-- PARTS -->
     <link name="robot_footprint"></link>
     <joint name="robot_footprint_joint" type="fixed">

File: src/myrobot_gazebo/urdf/myrobot_wheel.urdf.xacro (robot description, xacro)
@@ -1,4 +1,4 @@
 <?xml version="1.0"?>
-<robot xmlns:xacro="http://ros.org/wiki/xacro" name="husky_wheel">
+<robot xmlns:xacro="http://ros.org/wiki/xacro" name="myrobot_wheel">
 	<xacro:macro name="myrobot_wheel" params="wheel_prefix *joint_pose">
 		<link name="${wheel_prefix}_wheel">

Commit message: Fixed rotation issue by changing friction model. Tuned AMCL parameters to optimise.

File: src/myrobot_gazebo/urdf/myrobot.urdf.xacro (robot description, xacro)
@@ -6,12 +6,14 @@
     <!-- PROPERTIES -->
     <xacro:property name="M_PI" value="3.14159"/>
+    <xacro:property name="chassis_mass" value="15.0" />
     <xacro:property name="chassis_height" value="0.12" />
     <xacro:property name="chassis_length" value="0.4" />
-    <xacro:property name="chassis_width" value="0.25" />
+    <xacro:property name="chassis_width" value="0.2" />
+    <xacro:property name="wheel_mass" value="1.5" />
     <xacro:property name="wheel_width" value="0.06" />
     <xacro:property name="wheel_rad" value="0.1" />
     <xacro:property name="wheel_forward_offset" value="0.13" />
     <xacro:property name="wheel_left_offset" value="${chassis_width/2 + 0.05}" />
-    <xacro:property name="wheel_friction" value="0.3" />
+    <!-- <xacro:property name="wheel_friction" value="0.3" /> -->
     <xacro:property name="use_drive_controller" value="true" />
     <!-- PLUGINS -->
@@ -27,7 +29,12 @@
         <!-- <pose>0 0 0.1 0 0 0</pose> -->
         <inertial>
-            <mass value="15.0"/>
+            <mass value="${chassis_mass}"/>
             <origin xyz="0 0 0" rpy=" 0 0 0"/>
-            <inertia ixx="0.1" ixy="0" ixz="0" iyy="0.1" iyz="0" izz="0.1" />
+            <inertia    ixx="${1/12 * chassis_mass * (chassis_height**2 + chassis_width**2)}"
+                        ixy="0"
+                        ixz="0"
+                        iyy="${1/12 * chassis_mass * (chassis_height**2 + chassis_length**2)}"
+                        iyz="0"
+                        izz="${1/12 * chassis_mass * (chassis_length**2 + chassis_width**2)}" />
         </inertial>
         <collision name='collision'>

File: src/myrobot_gazebo/urdf/myrobot_wheel.urdf.xacro (robot description, xacro)
@@ -4,8 +4,13 @@
 		<link name="${wheel_prefix}_wheel">
 			<inertial>
-				<mass value="1.5" />
+				<mass value="${wheel_mass}" />
 				<!-- <origin xyz="0.0 0.0 0.0" rpy="0 ${M_PI/2} ${M_PI/2}"/> -->
 				<origin xyz="0.0 0.0 0.0" rpy="0 0 0"/>
-				<inertia ixx="0.005" ixy="0.0" ixz="0.0" iyy="0.005" iyz="0.0" izz="0.005"/>
+				<inertia 	ixx="${1/12 * wheel_mass * (3 * wheel_rad**2 + wheel_width**2)}"
+							ixy="0.0"
+							ixz="0.0"
+							iyy="${0.5 * wheel_mass * wheel_rad**2}"
+							iyz="0.0"
+							izz="${1/12 * wheel_mass * (3 * wheel_rad**2 + wheel_width**2)}" />
 			</inertial>
 			<visual name="${wheel_prefix}_wheel_visual">
@@ -24,8 +29,8 @@
             <visual name='front_left_wheel_bump'>
 				<xacro:if value="${wheel_prefix.endswith('left')}">
-                	<origin xyz="0.05 0.03 0.05" rpy=" 0 0 0"/>
+                	<origin xyz="${wheel_rad/2} 0.02 ${wheel_rad/2}" rpy=" 0 0 0"/>
 				</xacro:if>
 				<xacro:unless value="${wheel_prefix.endswith('left')}">
-                	<origin xyz="0.05 -0.03 0.05" rpy=" 0 0 0"/>
+                	<origin xyz="${wheel_rad/2} -0.02 ${wheel_rad/2}" rpy=" 0 0 0"/>
 				</xacro:unless>
                 <geometry>
@@ -35,9 +40,9 @@
 		</link>
 		<gazebo reference="${wheel_prefix}_wheel">
-			<mu1 value="1"/>
-			<mu2 value="1"/>
-			<kp value="10000000.0" />
-			<kd value="1.0" />
-			<fdir1 value="1 0 0"/>
+			<mu1 value="0.9"/>
+			<mu2 value="0.9"/>
+			<kp value="1000000.0" />
+			<kd value="10.0" />
+			<!-- <fdir1 value="0 0 1"/> -->
 		</gazebo>
 		<joint name="${wheel_prefix}_wheel_joint" type="continuous">
